File: hardware/nucleo-adapter/kicad/adapter.kicad_sch (KiCad schematic)
At the start: 103 parts, among them J1 Track +, J10 Motor A phase V, J11 Motor A phase W, J12 Nucleo PA15 (HIN1, motor B), J13 Nucleo PB8 (HIN2, motor B), J14 Nucleo PB9 (HIN3, motor B), J15 Nucleo PB3 (LIN1, motor B), J16 Nucleo PB4 (LIN2, motor B), J17 Nucleo PB5 (LIN3, motor B), J18 Motor B phase U, J19 Motor B phase V, J2 Track -, J20 Motor B phase W, J3 Nucleo PA8 (HIN1, motor A), J4 Nucleo PA9 (HIN2, motor A), J5 Nucleo PA10 (HIN3, motor A), J6 Nucleo PA7 (LIN1, motor A), J7 Nucleo PB0 (LIN2, motor A), J8 Nucleo PF0 (LIN3, motor A), J9 Motor A phase U, Q1 CSD16327Q3, Q10 CSD16327Q3 (high V, motor B), Q11 CSD16327Q3 (low V, motor B), Q12 CSD16327Q3 (high W, motor B), Q13 CSD16327Q3 (low W, motor B), Q2 CSD16327Q3 (high U, motor A), Q3 CSD16327Q3 (low U, motor A), Q4 CSD16327Q3 (high V, motor A), Q5 CSD16327Q3 (low V, motor A), Q6 CSD16327Q3 (high W, motor A), Q7 CSD16327Q3 (low W, motor A), Q8 CSD16327Q3 (high U, motor B), Q9 CSD16327Q3 (low U, motor B), U1 AP3012, U2 AP2204K-3.3, U3 MCP6002-xSN, U4 DRV8300D (motor A), U5 INA180A2, U6 DRV8300D (motor B), U7 INA180A2

Commit message: Clean up adapter schematic layout for readability, fix shunt topology bug
Layout: spread out the shared front end and both motor blocks with much
more generous spacing; paper bumped to A0 (drawing is ~470x410mm, too
big for A3/A1). Every pin now gets a short stub wire before its label
lands rather than the label sitting directly on the pin tip - needed
because several parts (AP3012, DRV8300D, CSD16327Q3) have multiple pins
within a few mm of each other on the symbol body itself. Genuinely-
unused pins (AP2204K-3.3 and DRV8300D's NC pins) get a proper no_connect
marker instead of a dangling stub. Simplified per-instance Value strings
so all 13 CSD16327Q3 FETs group into one BOM line instead of 12.

While untangling an overlapping label on the shared current-sense shunt,
found the bridges' high-side FET drains were wired to VBUS (pre-shunt)
instead of VBUS_LOAD (post-shunt) - the shunt was bypassed by the actual
load current entirely, contradicting DESIGN.md's own documented intent.
Fixed. Still 0 ERC errors.

Co-Authored-By: Claude Sonnet 5 <noreply@anthropic.com>
Parts:
- Q10: value CSD16327Q3 (high V, motor B) -> CSD16327Q3
- Q11: value CSD16327Q3 (low V, motor B) -> CSD16327Q3
- Q12: value CSD16327Q3 (high W, motor B) -> CSD16327Q3
- Q13: value CSD16327Q3 (low W, motor B) -> CSD16327Q3
- Q2: value CSD16327Q3 (high U, motor A) -> CSD16327Q3
- Q3: value CSD16327Q3 (low U, motor A) -> CSD16327Q3
- Q4: value CSD16327Q3 (high V, motor A) -> CSD16327Q3
- Q5: value CSD16327Q3 (low V, motor A) -> CSD16327Q3
- Q6: value CSD16327Q3 (high W, motor A) -> CSD16327Q3
- Q7: value CSD16327Q3 (low W, motor A) -> CSD16327Q3
- Q8: value CSD16327Q3 (high U, motor B) -> CSD16327Q3
- Q9: value CSD16327Q3 (low U, motor B) -> CSD16327Q3
- U4: value DRV8300D (motor A) -> DRV8300D (A)
- U6: value DRV8300D (motor B) -> DRV8300D (B)
Connections:
- net TRACK_PWR: no longer Q10.5 (D), Q12.5 (D), Q2.5 (D), Q4.5 (D), Q6.5 (D), Q8.5 (D), R4.2, R8.1
- new net VBUS_LOAD: Q10.5 (D), Q12.5 (D), Q2.5 (D), Q4.5 (D), Q6.5 (D), Q8.5 (D), R4.2, R8.1
- no-connect marks 0 -> 5
