File: hardware/nucleo-adapter/kicad/main.kicad_sch (KiCad schematic)
At the start: 1 part, among them U8 Nucleo-G474RE

Commit message: Place real Nucleo-G474RE symbol and fold it into the project libraries
Replaces the hand-authored black-box Nucleo block with the genuine
STMicroelectronics/SnapEDA symbol, wired by real CN7/CN10 pin number
rather than guessed pin names, and routed through dedicated lanes since
the real pinout doesn't line up with the sheets' pin order the way the
old placeholder did.

The symbol and its footprint were previously loose, unregistered files
(the footprint's library nickname didn't even exist in fp-lib-table).
Both now live inside the project's registered AdapterSymbols.kicad_sym
and AdapterFootprints.pretty libraries, referenced accordingly.

Co-Authored-By: Claude Sonnet 5 <noreply@anthropic.com>
Parts:
- removed U8: Nucleo-G474RE, symbol Local:Nucleo_G474RE
- added U8: (no value), symbol AdapterSymbols:NUCLEO-G474RE
Connections:
- net Motor A/GND: now also U8.CN7_19 (GND_CN7_19)
- net Motor A/PA0: now also U8.CN7_28 (PA0)
- net Motor A/PA1: now also U8.CN7_29 (PF0), U8.CN7_30 (PA1)
- net Motor A/PA10: now also U8.CN10_33 (PA10)
- net Motor A/PA3: now also U8.CN10_37 (PA3/PC5)
- net Motor A/PA7: now also U8.CN10_15 (PA7), U8.CN10_16 (PB12)
- net Motor A/PA8: now also U8.CN10_23 (PA8), U8.CN10_24 (PB1)
- net Motor A/PA9: now also U8.CN10_21 (PA9)
- net Motor A/PB0: now also U8.CN7_34 (PB0)
- net Motor A/PB11: now also U8.CN10_18 (PB11)
- net Motor A/VDD: now also U8.CN7_16 (+3V3)
- net Motor B/PA15: now also U8.CN7_17 (PA15)
- net Motor B/PA4: now also U8.CN7_31 (PF1), U8.CN7_32 (PA4)
- net Motor B/PA5: now also U8.CN10_11 (PA5)
- net Motor B/PA6: now also U8.CN10_13 (PA6)
- net Motor B/PB14: now also U8.CN10_27 (PB4), U8.CN10_28 (PB14)
- net Motor B/PB3: now also U8.CN10_31 (PB3)
- net Motor B/PB5: now also U8.CN10_29 (PB5)
- net Motor B/PB8: now also U8.CN10_3 (PB8)
- net Motor B/PB9: now also U8.CN10_5 (PB9)
- net Power/PA2: now also U8.CN10_35 (PA2/PC4)
- no-connect marks 0 -> 50
