File: hardware/RemoraNextGen/RemoraNextGen.kicad_sch (KiCad schematic)
At the start: 1 part, among them U8 Nucleo-G474RE

Commit message: Fit sub-sheet blocks on the page; wire local nets in power schematic
Motor B's sheet box ran from y=610 to y=1010, but the A0 landscape root
page is only 841mm tall - it silently overflowed the bottom edge by
169mm. Motor A/B's box heights (400mm) were also far bigger than their
actual pin content needs (~240mm). Tightened both to 260mm and now
compute each sheet's Y position from the previous one's bottom edge
plus a fixed gap, instead of hardcoded absolute numbers, so this can't
drift out of sync with the page again.

finalize_nets() previously only drew a real wire for nets with exactly
2 points, so every net touched at 3+ points - the majority of the
power schematic - stayed as disconnected floating labels. Now any net
whose points stay within a 150mm span gets chained together with real
wire regardless of point count; only genuinely page-wide rails (GND,
VCC, VDD, VBUS, and similarly wide-spanning nets like a motor's phase
node or return net) still fall back to labels, matching how a real
schematic handles shared rails. Verified motor_a/b's wide nets still
correctly fall back to labels rather than turning into a new rats-nest.

ERC still 0 errors throughout.

Also ignores ~*.lck (KiCad's file-open lock markers).

Co-Authored-By: Claude Sonnet 5 <noreply@anthropic.com>
Changed lines of the file:
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@@
 	(sheet
 		(at 354.00 170.00)
-		(size 140.00 400.00)
+		(size 140.00 260.00)
 		(exclude_from_sim no)
 		(in_bom yes)
@@
 		(fill (color 0 0 0 0))
 		(property "Sheetname" "Motor A" (at 354.00 167.00 0) (effects (font (size 1.27 1.27)) (justify left bottom)))
-		(property "Sheetfile" "motor_a.kicad_sch" (at 354.00 573.00 0) (effects (font (size 1.27 1.27)) (justify left top)))
+		(property "Sheetfile" "motor_a.kicad_sch" (at 354.00 433.00 0) (effects (font (size 1.27 1.27)) (justify left top)))
 		(pin "VCC" input (at 354.00 185.00 180) (effects (font (size 1.27 1.27))))
 		(pin "VDD" input (at 354.00 200.00 180) (effects (font (size 1.27 1.27))))
@@
 	)
 	(sheet
-		(at 354.00 610.00)
-		(size 140.00 400.00)
+		(at 354.00 450.00)
+		(size 140.00 260.00)
 		(exclude_from_sim no)
 		(in_bom yes)
@@
 		(stroke (width 0.1524) (type solid))
 		(fill (color 0 0 0 0))
-		(property "Sheetname" "Motor B" (at 354.00 607.00 0) (effects (font (size 1.27 1.27)) (justify left bottom)))
-		(property "Sheetfile" "motor_b.kicad_sch" (at 354.00 1013.00 0) (effects (font (size 1.27 1.27)) (justify left top)))
-		(pin "VCC" input (at 354.00 625.00 180) (effects (font (size 1.27 1.27))))
-		(pin "VDD" input (at 354.00 640.00 180) (effects (font (size 1.27 1.27))))
-		(pin "GND" passive (at 354.00 655.00 180) (effects (font (size 1.27 1.27))))
-		(pin "VBUS_LOAD" input (at 354.00 670.00 180) (effects (font (size 1.27 1.27))))
-		(pin "PA15" input (at 354.00 700.00 180) (effects (font (size 1.27 1.27))))
-		(pin "PB8" input (at 354.00 715.00 180) (effects (font (size 1.27 1.27))))
-		(pin "PB9" input (at 354.00 730.00 180) (effects (font (size 1.27 1.27))))
-		(pin "PB3" input (at 354.00 745.00 180) (effects (font (size 1.27 1.27))))
-		(pin "PB4" input (at 354.00 760.00 180) (effects (font (size 1.27 1.27))))
-		(pin "PB5" input (at 354.00 775.00 180) (effects (font (size 1.27 1.27))))
-		(pin "PA4" output (at 354.00 790.00 180) (effects (font (size 1.27 1.27))))
-		(pin "PA5" output (at 354.00 805.00 180) (effects (font (size 1.27 1.27))))
-		(pin "PA6" output (at 354.00 820.00 180) (effects (font (size 1.27 1.27))))
-		(pin "PB14" output (at 354.00 835.00 180) (effects (font (size 1.27 1.27))))
-		(pin "PF1" output (at 354.00 850.00 180) (effects (font (size 1.27 1.27))))
+		(property "Sheetname" "Motor B" (at 354.00 447.00 0) (effects (font (size 1.27 1.27)) (justify left bottom)))
+		(property "Sheetfile" "motor_b.kicad_sch" (at 354.00 713.00 0) (effects (font (size 1.27 1.27)) (justify left top)))
+		(pin "VCC" input (at 354.00 465.00 180) (effects (font (size 1.27 1.27))))
+		(pin "VDD" input (at 354.00 480.00 180) (effects (font (size 1.27 1.27))))
+		(pin "GND" passive (at 354.00 495.00 180) (effects (font (size 1.27 1.27))))
+		(pin "VBUS_LOAD" input (at 354.00 510.00 180) (effects (font (size 1.27 1.27))))
+		(pin "PA15" input (at 354.00 540.00 180) (effects (font (size 1.27 1.27))))
+		(pin "PB8" input (at 354.00 555.00 180) (effects (font (size 1.27 1.27))))
+		(pin "PB9" input (at 354.00 570.00 180) (effects (font (size 1.27 1.27))))
+		(pin "PB3" input (at 354.00 585.00 180) (effects (font (size 1.27 1.27))))
+		(pin "PB4" input (at 354.00 600.00 180) (effects (font (size 1.27 1.27))))
+		(pin "PB5" input (at 354.00 615.00 180) (effects (font (size 1.27 1.27))))
+		(pin "PA4" output (at 354.00 630.00 180) (effects (font (size 1.27 1.27))))
+		(pin "PA5" output (at 354.00 645.00 180) (effects (font (size 1.27 1.27))))
+		(pin "PA6" output (at 354.00 660.00 180) (effects (font (size 1.27 1.27))))
+		(pin "PB14" output (at 354.00 675.00 180) (effects (font (size 1.27 1.27))))
+		(pin "PF1" output (at 354.00 690.00 180) (effects (font (size 1.27 1.27))))
 		(instances (project "RemoraNextGen" (path "/10000000-0000-0000-0000-000000000001" (page "4"))))
 	)
@@
 	)
 	(wire
-		(pts (xy 252.00 187.46) (xy 252.00 700.00))
-		(stroke (width 0) (type default))
-	)
-	(wire
-		(pts (xy 252.00 700.00) (xy 354.00 700.00))
+		(pts (xy 252.00 187.46) (xy 252.00 540.00))
+		(stroke (width 0) (type default))
+	)
+	(wire
+		(pts (xy 252.00 540.00) (xy 354.00 540.00))
 		(stroke (width 0) (type default))
 	)
@@
 	)
 	(wire
-		(pts (xy 258.00 279.68) (xy 258.00 715.00))
-		(stroke (width 0) (type default))
-	)
-	(wire
-		(pts (xy 258.00 715.00) (xy 354.00 715.00))
+		(pts (xy 258.00 279.68) (xy 258.00 555.00))
+		(stroke (width 0) (type default))
+	)
+	(wire
+		(pts (xy 258.00 555.00) (xy 354.00 555.00))
 		(stroke (width 0) (type default))
 	)
@@
 	)
 	(wire
-		(pts (xy 264.00 282.22) (xy 264.00 730.00))
-		(stroke (width 0) (type default))
-	)
-	(wire
-		(pts (xy 264.00 730.00) (xy 354.00 730.00))
+		(pts (xy 264.00 282.22) (xy 264.00 570.00))
+		(stroke (width 0) (type default))
+	)
+	(wire
+		(pts (xy 264.00 570.00) (xy 354.00 570.00))
 		(stroke (width 0) (type default))
 	)
@@
 	)
 	(wire
-		(pts (xy 270.00 315.24) (xy 270.00 745.00))
-		(stroke (width 0) (type default))
-	)
-	(wire
-		(pts (xy 270.00 745.00) (xy 354.00 745.00))
+		(pts (xy 270.00 315.24) (xy 270.00 585.00))
+		(stroke (width 0) (type default))
+	)
+	(wire
+		(pts (xy 270.00 585.00) (xy 354.00 585.00))
 		(stroke (width 0) (type default))
 	)
@@
 	)
 	(wire
-		(pts (xy 276.00 310.16) (xy 276.00 760.00))
-		(stroke (width 0) (type default))
-	)
-	(wire
-		(pts (xy 276.00 760.00) (xy 354.00 760.00))
+		(pts (xy 276.00 310.16) (xy 276.00 600.00))
+		(stroke (width 0) (type default))
+	)
+	(wire
+		(pts (xy 276.00 600.00) (xy 354.00 600.00))
 		(stroke (width 0) (type default))
 	)
@@
 	)
 	(wire
-		(pts (xy 282.00 312.70) (xy 282.00 775.00))
-		(stroke (width 0) (type default))
-	)
-	(wire
-		(pts (xy 282.00 775.00) (xy 354.00 775.00))
+		(pts (xy 282.00 312.70) (xy 282.00 615.00))
+		(stroke (width 0) (type default))
+	)
+	(wire
+		(pts (xy 282.00 615.00) (xy 354.00 615.00))
 		(stroke (width 0) (type default))
 	)
@@
 	)
 	(wire
-		(pts (xy 288.00 205.24) (xy 288.00 790.00))
-		(stroke (width 0) (type default))
-	)
-	(wire
-		(pts (xy 288.00 790.00) (xy 354.00 790.00))
+		(pts (xy 288.00 205.24) (xy 288.00 630.00))
+		(stroke (width 0) (type default))
+	)
+	(wire
+		(pts (xy 288.00 630.00) (xy 354.00 630.00))
 		(stroke (width 0) (type default))
 	)
@@
 	)
 	(wire
-		(pts (xy 294.00 289.84) (xy 294.00 805.00))
-		(stroke (width 0) (type default))
-	)
-	(wire
-		(pts (xy 294.00 805.00) (xy 354.00 805.00))
+		(pts (xy 294.00 289.84) (xy 294.00 645.00))
+		(stroke (width 0) (type default))
+	)
+	(wire
+		(pts (xy 294.00 645.00) (xy 354.00 645.00))
 		(stroke (width 0) (type default))
 	)
@@
 	)
 	(wire
-		(pts (xy 300.00 292.38) (xy 300.00 820.00))
-		(stroke (width 0) (type default))
-	)
-	(wire
-		(pts (xy 300.00 820.00) (xy 354.00 820.00))
+		(pts (xy 300.00 292.38) (xy 300.00 660.00))
+		(stroke (width 0) (type default))
+	)
+	(wire
+		(pts (xy 300.00 660.00) (xy 354.00 660.00))
 		(stroke (width 0) (type default))
 	)
@@
 	)
 	(wire
-		(pts (xy 306.00 310.16) (xy 306.00 835.00))
-		(stroke (width 0) (type default))
-	)
-	(wire
-		(pts (xy 306.00 835.00) (xy 354.00 835.00))
+		(pts (xy 306.00 310.16) (xy 306.00 675.00))
+		(stroke (width 0) (type default))
+	)
+	(wire
+		(pts (xy 306.00 675.00) (xy 354.00 675.00))
 		(stroke (width 0) (type default))
 	)
@@
 	)
 	(wire
-		(pts (xy 312.00 205.24) (xy 312.00 850.00))
-		(stroke (width 0) (type default))
-	)
-	(wire
-		(pts (xy 312.00 850.00) (xy 354.00 850.00))
+		(pts (xy 312.00 205.24) (xy 312.00 690.00))
+		(stroke (width 0) (type default))
+	)
+	(wire
+		(pts (xy 312.00 690.00) (xy 354.00 690.00))
 		(stroke (width 0) (type default))
 	)
@@
 	)
 	(wire
-		(pts (xy 524.00 185.00) (xy 524.00 625.00))
-		(stroke (width 0) (type default))
-	)
-	(wire
-		(pts (xy 524.00 625.00) (xy 354.00 625.00))
+		(pts (xy 524.00 185.00) (xy 524.00 465.00))
+		(stroke (width 0) (type default))
+	)
+	(wire
+		(pts (xy 524.00 465.00) (xy 354.00 465.00))
 		(stroke (width 0) (type default))
 	)
@@
 	)
 	(wire
-		(pts (xy 534.00 200.00) (xy 534.00 640.00))
-		(stroke (width 0) (type default))
-	)
-	(wire
-		(pts (xy 534.00 640.00) (xy 354.00 640.00))
+		(pts (xy 534.00 200.00) (xy 534.00 480.00))
+		(stroke (width 0) (type default))
+	)
+	(wire
+		(pts (xy 534.00 480.00) (xy 354.00 480.00))
 		(stroke (width 0) (type default))
 	)
@@
 	)
 	(wire
-		(pts (xy 544.00 215.00) (xy 544.00 655.00))
-		(stroke (width 0) (type default))
-	)
-	(wire
-		(pts (xy 544.00 655.00) (xy 354.00 655.00))
+		(pts (xy 544.00 215.00) (xy 544.00 495.00))
+		(stroke (width 0) (type default))
+	)
+	(wire
+		(pts (xy 544.00 495.00) (xy 354.00 495.00))
 		(stroke (width 0) (type default))
 	)
@@
 	)
 	(wire
-		(pts (xy 554.00 230.00) (xy 554.00 670.00))
-		(stroke (width 0) (type default))
-	)
-	(wire
-		(pts (xy 554.00 670.00) (xy 354.00 670.00))
-		(stroke (width 0) (type default))
-	)
+		(pts (xy 554.00 230.00) (xy 554.00 510.00))
+		(stroke (width 0) (type default))
+	)
+	(wire
+		(pts (xy 554.00 510.00) (xy 354.00 510.00))
+		(stroke (width 0) (type default))
+	)
